File: SPROJ2_G3_PCB.kicad_sch (KiCad schematic)
At the start: 87 parts, among them IC1 TPS61175PWPR, J10 Conn_01x02_Pin, J11 Conn_01x05_Pin, J12 Conn_01x03_Pin, J13 Conn_01x02_Pin, J14 UJC-HP-3-SMT-TR, J4 Conn_01x03_Pin, J5 Conn_01x02_Pin, J6 Conn_01x02_Pin, J7 Conn_01x02_Pin, J9 Conn_01x02_Pin, P1 5k, P2 R_Potentiometer, Q1 Q_NMOS_GSD, Q2 Q_PMOS_GSD, U1 LMV324, U2 LMV324, U5 MCP73831T-2ACI_OT, U7 MC7805CDTG, Y1 Crystal

Commit message: Add files via upload
Parts:
- removed LCD1: Conn_01x04_Pin, Connector_JST:JST_PH_S4B-PH-K_1x04_P2.00mm_Horizontal, symbol Connector:Conn_01x04_Pin
- removed P2: R_Potentiometer, Potentiometer_THT:Potentiometer_ACP_CA6-H2,5_Horizontal, symbol Device:R_Potentiometer
- added R38: 39k, symbol Device:R
- added R39: 10k, symbol Device:R
- C17: value 22u -> 470u
- C18: value 0.33u -> 470n
- R13: value 1k -> 910
- R17: value 59k -> 56k
- R18: value 909 -> 910
- R36, R37: value 51k -> 100k
- R? (x2): value 10k -> 100k
Connections:
- net +5V: now also R38.1; no longer R32.2
- net Feedback: now also IC1.9 (FB); no longer IC1.10 (FREQ), R17.2
- net GND: now also R39.2
- net PI_EN: no longer Q2.1 (G)
- net POT_1: no longer P1.1, P1.2
- net at J12.1 (Pin_1), R33.1: no longer Q2.2 (S), Q2.3 (D)
- net at U1.13 (-): now also R38.2, R39.1
- new net: IC1.10 (FREQ), R17.2
- no-connect marks 3 -> 9
Other:
- note added: "1st Stage Filters: - Passive HPF: fc = 0.5Hz - Active LPF: fc = 3.4Hz - Non-inverting Amplifier: Gain 1001x"
- note added: "2nd Order Active Butterworth LPF -40dB @ 50Hz"
- note added: "2nd Stage Filters"
- note added: "5V Linear Voltage Regulator"
- note added: "Block 1 Battery Management System"
- note added: "Block 2 DC-DC Boost Converter circuit"
- note added: "Block 3 Temperature measurement schematic"
- note added: "Block 4 Atmel ATmega 328P microcontroller"
- note added: "Block 5 Connectors"
- note added: "Block 6 Pulse sensing schematic"
- note added: "Block 7 Redundancy system"
- note added: "Comparator"
- note added: "Current limiting with Op-amp"
- note added: "Differential Buffer"
- note added: "External Pulse Sensor"
- note added: "LM75 temperature sensor"
- note added: "NTC connector"
- note added: "Non-inverting Amplifier 6.6x Gain"
- note added: "OLED Display"
- note added: "Pull-up resistors for the I2C data lines"
- note added: "Reconfigured due to not being in use"
- note added: "TCRT1000 optical sensor"
- note added: "Wheatstone Bridge"
- note removed: "Block_1 (Battery + USB_C)"
- note removed: "Block_2 (NMOS + DC to DC)"
- note removed: "Block_3 (Temperature)"
- note removed: "Block_4 (Atmega)"
- note removed: "Block_5 (Connectors)"
- note removed: "Block_6 (Pulse Sensor)"
- note removed: "Block_7 (Redundancy system)"
- note removed: "Display"
- note removed: "LM75"
- note removed: "NTC"
- note removed: "PULSE"
- note removed: "PUll-up"
- moved on the sheet: J4, R24, R25, R32, R36, R37, U1C

Commit message: Add files via upload
Parts:
- R38: value 39k -> 390k
- R39: value 10k -> 100k
- renumbered R32 to R32*, R35 to R35*
Connections:
- net +5V: now also C17.1, C20.2, D1.1 (K), L2.1, R15.2, R36.2; no longer C20.1, R36.1
- net GND: now also C20.1, R32*.2; no longer C20.2
- net Non_INV_C_1: now also R36.1; no longer R36.2
- net PI_EN: now also Q2.1 (G)
- net at R38.2, R39.1, U1.13 (-): now also R35*.2
- no-connect marks 9 -> 6
Other:
- moved on the sheet: C12, C17, C20, C21, C4, C5, C8, C9, D2, FTDI1, J4, LCD1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

Commit message: Final sch
Final sch
Parts:
- C17: value 470u -> 220u
- L_5.6: value 5.6 -> 5.6u
- R17: value 56k -> 120k
Changed lines of the file:
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@@
 			)
 		)
-		(property "Value" "470u"
+		(property "Value" "220u"
 			(at 93.599 126.873 0)
 			(effects
@@
 			)
 		)
-		(property "Value" "56k"
-			(at 83.185 145.415 0)
+		(property "Value" "120k"
+			(at 83.312 147.32 0)
 			(effects
 				(font
@@
 			)
 		)
-		(property "Value" "5.6"
+		(property "Value" "5.6u"
 			(at 59.69 105.41 0)
 			(effects
